File: Test_boards/Led_tests/Led_tests.sch (KiCad schematic (older format))
At the start: 13 parts, among them J1 Screw_Terminal_01x02

Commit message: Completed LED castellated hole test board
Parts:
- D1: value LED -> 3.0mm; footprint (none) -> LTST-S110KGKT_castellated:LTST-S110KGKT_castellated_3.0mm
- D2: value LED -> 3.1mm; footprint (none) -> LTST-S110KGKT_castellated:LTST-S110KGKT_castellated_3.1mm
- D3: value LED -> 3.2mm; footprint (none) -> LTST-S110KGKT_castellated:LTST-S110KGKT_castellated_3.2mm
- D4: value LED -> 3.3mm; footprint (none) -> LTST-S110KGKT_castellated:LTST-S110KGKT_castellated_3.3mm
- D5: value LED -> 3.4mm; footprint (none) -> LTST-S110KGKT_castellated:LTST-S110KGKT_castellated_3.4mm
- D6: value LED -> 3.5mm; footprint (none) -> LTST-S110KGKT_castellated:LTST-S110KGKT_castellated_3.5mm
- J1: footprint (none) -> TerminalBlock:TerminalBlock_bornier-2_P5.08mm
- RN1, RN2, RN3, RN4, RN5, RN6: footprint (none) -> Resistor_SMD:R_Array_Concave_4x0603
Changed lines of the file:
@@
 EESchema Schematic File Version 4
+LIBS:Led_tests-cache
 EELAYER 26 0
 EELAYER END
@@
 P 1500 1850
 F 0 "D1" V 1538 1733 50  0000 R CNN
-F 1 "LED" V 1447 1733 50  0000 R CNN
-F 2 "" H 1500 1850 50  0001 C CNN
+F 1 "3.0mm" V 1447 1733 50  0000 R CNN
+F 2 "LTST-S110KGKT_castellated:LTST-S110KGKT_castellated_3.0mm" H 1500 1850 50  0001 C CNN
 F 3 "~" H 1500 1850 50  0001 C CNN
 	1    1500 1850
@@
 F 0 "RN1" H 1738 1446 50  0000 L CNN
 F 1 "R_Pack04" H 1738 1355 50  0000 L CNN
-F 2 "" V 1825 1400 50  0001 C CNN
+F 2 "Resistor_SMD:R_Array_Concave_4x0603" V 1825 1400 50  0001 C CNN
 F 3 "~" H 1550 1400 50  0001 C CNN
 	1    1550 1400
@@
 P 1500 2950
 F 0 "D2" V 1538 2833 50  0000 R CNN
-F 1 "LED" V 1447 2833 50  0000 R CNN
-F 2 "" H 1500 2950 50  0001 C CNN
+F 1 "3.1mm" V 1447 2833 50  0000 R CNN
+F 2 "LTST-S110KGKT_castellated:LTST-S110KGKT_castellated_3.1mm" H 1500 2950 50  0001 C CNN
 F 3 "~" H 1500 2950 50  0001 C CNN
 	1    1500 2950
@@
 F 0 "RN2" H 1738 2546 50  0000 L CNN
 F 1 "R_Pack04" H 1738 2455 50  0000 L CNN
-F 2 "" V 1825 2500 50  0001 C CNN
+F 2 "Resistor_SMD:R_Array_Concave_4x0603" V 1825 2500 50  0001 C CNN
 F 3 "~" H 1550 2500 50  0001 C CNN
 	1    1550 2500
@@
 P 2400 1850
 F 0 "D3" V 2438 1733 50  0000 R CNN
-F 1 "LED" V 2347 1733 50  0000 R CNN
-F 2 "" H 2400 1850 50  0001 C CNN
+F 1 "3.2mm" V 2347 1733 50  0000 R CNN
+F 2 "LTST-S110KGKT_castellated:LTST-S110KGKT_castellated_3.2mm" H 2400 1850 50  0001 C CNN
 F 3 "~" H 2400 1850 50  0001 C CNN
 	1    2400 1850
@@
 F 0 "RN3" H 2638 1446 50  0000 L CNN
 F 1 "R_Pack04" H 2638 1355 50  0000 L CNN
-F 2 "" V 2725 1400 50  0001 C CNN
+F 2 "Resistor_SMD:R_Array_Concave_4x0603" V 2725 1400 50  0001 C CNN
 F 3 "~" H 2450 1400 50  0001 C CNN
 	1    2450 1400
@@
 P 2400 2950
 F 0 "D4" V 2438 2833 50  0000 R CNN
-F 1 "LED" V 2347 2833 50  0000 R CNN
-F 2 "" H 2400 2950 50  0001 C CNN
+F 1 "3.3mm" V 2347 2833 50  0000 R CNN
+F 2 "LTST-S110KGKT_castellated:LTST-S110KGKT_castellated_3.3mm" H 2400 2950 50  0001 C CNN
 F 3 "~" H 2400 2950 50  0001 C CNN
 	1    2400 2950
@@
 F 0 "RN4" H 2638 2546 50  0000 L CNN
 F 1 "R_Pack04" H 2638 2455 50  0000 L CNN
-F 2 "" V 2725 2500 50  0001 C CNN
+F 2 "Resistor_SMD:R_Array_Concave_4x0603" V 2725 2500 50  0001 C CNN
 F 3 "~" H 2450 2500 50  0001 C CNN
 	1    2450 2500
@@
 P 3300 1850
 F 0 "D5" V 3338 1733 50  0000 R CNN
-F 1 "LED" V 3247 1733 50  0000 R CNN
-F 2 "" H 3300 1850 50  0001 C CNN
+F 1 "3.4mm" V 3247 1733 50  0000 R CNN
+F 2 "LTST-S110KGKT_castellated:LTST-S110KGKT_castellated_3.4mm" H 3300 1850 50  0001 C CNN
 F 3 "~" H 3300 1850 50  0001 C CNN
 	1    3300 1850
@@
 F 0 "RN5" H 3538 1446 50  0000 L CNN
 F 1 "R_Pack04" H 3538 1355 50  0000 L CNN
-F 2 "" V 3625 1400 50  0001 C CNN
+F 2 "Resistor_SMD:R_Array_Concave_4x0603" V 3625 1400 50  0001 C CNN
 F 3 "~" H 3350 1400 50  0001 C CNN
 	1    3350 1400
@@
 P 3300 2950
 F 0 "D6" V 3338 2833 50  0000 R CNN
-F 1 "LED" V 3247 2833 50  0000 R CNN
-F 2 "" H 3300 2950 50  0001 C CNN
+F 1 "3.5mm" V 3247 2833 50  0000 R CNN
+F 2 "LTST-S110KGKT_castellated:LTST-S110KGKT_castellated_3.5mm" H 3300 2950 50  0001 C CNN
 F 3 "~" H 3300 2950 50  0001 C CNN
 	1    3300 2950
@@
 F 0 "RN6" H 3538 2546 50  0000 L CNN
 F 1 "R_Pack04" H 3538 2455 50  0000 L CNN
-F 2 "" V 3625 2500 50  0001 C CNN
+F 2 "Resistor_SMD:R_Array_Concave_4x0603" V 3625 2500 50  0001 C CNN
 F 3 "~" H 3350 2500 50  0001 C CNN
 	1    3350 2500
@@
 F 0 "J1" H 770 2075 50  0000 C CNN
 F 1 "Screw_Terminal_01x02" H 770 2166 50  0000 C CNN
-F 2 "" H 850 2400 50  0001 C CNN
+F 2 "TerminalBlock:TerminalBlock_bornier-2_P5.08mm" H 850 2400 50  0001 C CNN
 F 3 "~" H 850 2400 50  0001 C CNN
 	1    850  2400
