File: Test_boards/Cap_touch_test/Cap_touch_test.sch (KiCad schematic (older format))
At the start: 15 parts, among them J1 Conn_02x05_Odd_Even, J2 Screw_Terminal_01x02, U1 LPC804-TSSOP24

Commit message: saving progress.
Other:
- note added: "Note: KiCAD does not have Cap Touch pad support."
Changed lines of the file:
@@
 EESchema Schematic File Version 4
+LIBS:Cap_touch_test-cache
 EELAYER 26 0
 EELAYER END
@@
 Wire Wire Line
 	4350 2250 4150 2250
+Text Notes 2200 3650 0    50   ~ 0
+Note: KiCAD does not have Cap Touch pad support.
 $EndSCHEMATC

Commit message: Complicated pads are beyond my skills at the moment. I will need to create something of 'fill zones'. I reached out some feelers on hackaday but I am proceeding with my current information.
Parts:
- C1, C6, C7: footprint (none) -> Capacitor_SMD:C_0805_2012Metric
- D1, D2, D3, D4: footprint (none) -> Diode_SMD:D_0805_2012Metric
- J1: footprint (none) -> Connector_PinHeader_1.27mm:PinHeader_2x05_P1.27mm_Vertical
- J2: footprint (none) -> TerminalBlock:TerminalBlock_bornier-2_P5.08mm
- RN1: footprint (none) -> Resistor_SMD:R_Array_Concave_4x0603
- U1: footprint (none) -> Package_SO:TSSOP-24_4.4x7.8mm_P0.65mm
Changed lines of the file:
@@
 F 0 "U1" H 2950 2728 50  0000 C CNN
 F 1 "LPC804-TSSOP24" H 2950 2637 50  0000 C CNN
-F 2 "" H 2250 1900 50  0001 C CNN
+F 2 "Package_SO:TSSOP-24_4.4x7.8mm_P0.65mm" H 2250 1900 50  0001 C CNN
 F 3 "" H 2250 1900 50  0001 C CNN
 	1    2950 1900
@@
 F 0 "J2" H 5930 792 50  0000 L CNN
 F 1 "Screw_Terminal_01x02" H 5930 701 50  0000 L CNN
-F 2 "" H 5850 800 50  0001 C CNN
+F 2 "TerminalBlock:TerminalBlock_bornier-2_P5.08mm" H 5850 800 50  0001 C CNN
 F 3 "~" H 5850 800 50  0001 C CNN
 	1    5850 800
@@
 F 0 "C6" H 5578 1346 50  0000 L CNN
 F 1 "0.1uF" H 5578 1255 50  0000 L CNN
-F 2 "" H 5400 1300 50  0001 C CNN
+F 2 "Capacitor_SMD:C_0805_2012Metric" H 5400 1300 50  0001 C CNN
 F 3 "~" H 5400 1300 50  0001 C CNN
 	1    5400 1300
@@
 F 0 "C7" H 6178 1346 50  0000 L CNN
 F 1 "0.1uF" H 6178 1255 50  0000 L CNN
-F 2 "" H 6000 1300 50  0001 C CNN
+F 2 "Capacitor_SMD:C_0805_2012Metric" H 6000 1300 50  0001 C CNN
 F 3 "~" H 6000 1300 50  0001 C CNN
 	1    6000 1300
@@
 F 0 "J1" H 1100 2317 50  0000 C CNN
 F 1 "Conn_02x05_Odd_Even" H 1100 2226 50  0000 C CNN
-F 2 "" H 1050 1900 50  0001 C CNN
+F 2 "Connector_PinHeader_1.27mm:PinHeader_2x05_P1.27mm_Vertical" H 1050 1900 50  0001 C CNN
 F 3 "~" H 1050 1900 50  0001 C CNN
 	1    1050 1900
@@
 F 0 "RN1" H 5988 2096 50  0000 L CNN
 F 1 "R_Pack04" H 5988 2005 50  0000 L CNN
-F 2 "" V 6075 2050 50  0001 C CNN
+F 2 "Resistor_SMD:R_Array_Concave_4x0603" V 6075 2050 50  0001 C CNN
 F 3 "~" H 5800 2050 50  0001 C CNN
 	1    5800 2050
@@
 F 0 "D1" V 5346 2382 50  0000 R CNN
 F 1 "Red" V 5255 2382 50  0000 R CNN
-F 2 "" V 5300 2450 50  0001 C CNN
+F 2 "Diode_SMD:D_0805_2012Metric" V 5300 2450 50  0001 C CNN
 F 3 "~" V 5300 2450 50  0001 C CNN
 	1    5300 2450
@@
 F 0 "D2" V 5646 2382 50  0000 R CNN
 F 1 "Red" V 5555 2382 50  0000 R CNN
-F 2 "" V 5600 2450 50  0001 C CNN
+F 2 "Diode_SMD:D_0805_2012Metric" V 5600 2450 50  0001 C CNN
 F 3 "~" V 5600 2450 50  0001 C CNN
 	1    5600 2450
@@
 F 0 "D3" V 5946 2382 50  0000 R CNN
 F 1 "Red" V 5855 2382 50  0000 R CNN
-F 2 "" V 5900 2450 50  0001 C CNN
+F 2 "Diode_SMD:D_0805_2012Metric" V 5900 2450 50  0001 C CNN
 F 3 "~" V 5900 2450 50  0001 C CNN
 	1    5900 2450
@@
 F 0 "D4" V 6246 2382 50  0000 R CNN
 F 1 "Red" V 6155 2382 50  0000 R CNN
-F 2 "" V 6200 2450 50  0001 C CNN
+F 2 "Diode_SMD:D_0805_2012Metric" V 6200 2450 50  0001 C CNN
 F 3 "~" V 6200 2450 50  0001 C CNN
 	1    6200 2450
@@
 F 0 "C1" V 1335 3400 50  0000 C CNN
 F 1 "0.1uF" V 1426 3400 50  0000 C CNN
-F 2 "" H 1650 3400 50  0001 C CNN
+F 2 "Capacitor_SMD:C_0805_2012Metric" H 1650 3400 50  0001 C CNN
 F 3 "~" H 1650 3400 50  0001 C CNN
 	1    1650 3400

Commit message: Added test cap touch pads to test board. Added renders. Review before initial submission to PCBway for manufacturing.
Parts:
- C2, C3, C4, C5: footprint (none) -> cap_touch_LPC804_NXP:Cap_T_pad
Changed lines of the file:
@@
 F 0 "C2" H 2578 3196 50  0000 L CNN
 F 1 "CAPT" H 2578 3105 50  0000 L CNN
-F 2 "" H 2400 3150 50  0001 C CNN
+F 2 "cap_touch_LPC804_NXP:Cap_T_pad" H 2400 3150 50  0001 C CNN
 F 3 "~" H 2400 3150 50  0001 C CNN
 	1    2400 3150
@@
 F 0 "C3" H 3228 3196 50  0000 L CNN
 F 1 "CAPT" H 3228 3105 50  0000 L CNN
-F 2 "" H 3050 3150 50  0001 C CNN
+F 2 "cap_touch_LPC804_NXP:Cap_T_pad" H 3050 3150 50  0001 C CNN
 F 3 "~" H 3050 3150 50  0001 C CNN
 	1    3050 3150
@@
 F 0 "C4" H 3828 3196 50  0000 L CNN
 F 1 "CAPT" H 3828 3105 50  0000 L CNN
-F 2 "" H 3650 3150 50  0001 C CNN
+F 2 "cap_touch_LPC804_NXP:Cap_T_pad" H 3650 3150 50  0001 C CNN
 F 3 "~" H 3650 3150 50  0001 C CNN
 	1    3650 3150
@@
 F 0 "C5" H 4428 3196 50  0000 L CNN
 F 1 "CAPT" H 4428 3105 50  0000 L CNN
-F 2 "" H 4250 3150 50  0001 C CNN
+F 2 "cap_touch_LPC804_NXP:Cap_T_pad" H 4250 3150 50  0001 C CNN
 F 3 "~" H 4250 3150 50  0001 C CNN
 	1    4250 3150

Commit message: Test boards submitted to PCBway for review and approval.
Parts:
- C2, C3, C4, C5: footprint cap_touch_LPC804_NXP:Cap_T_pad -> cap_touch_LPC804_NXP:Cap_T_pad_v1.1
Changed lines of the file:
@@
 F 0 "C2" H 2578 3196 50  0000 L CNN
 F 1 "CAPT" H 2578 3105 50  0000 L CNN
-F 2 "cap_touch_LPC804_NXP:Cap_T_pad" H 2400 3150 50  0001 C CNN
+F 2 "cap_touch_LPC804_NXP:Cap_T_pad_v1.1" H 2400 3150 50  0001 C CNN
 F 3 "~" H 2400 3150 50  0001 C CNN
 	1    2400 3150
@@
 F 0 "C3" H 3228 3196 50  0000 L CNN
 F 1 "CAPT" H 3228 3105 50  0000 L CNN
-F 2 "cap_touch_LPC804_NXP:Cap_T_pad" H 3050 3150 50  0001 C CNN
+F 2 "cap_touch_LPC804_NXP:Cap_T_pad_v1.1" H 3050 3150 50  0001 C CNN
 F 3 "~" H 3050 3150 50  0001 C CNN
 	1    3050 3150
@@
 F 0 "C4" H 3828 3196 50  0000 L CNN
 F 1 "CAPT" H 3828 3105 50  0000 L CNN
-F 2 "cap_touch_LPC804_NXP:Cap_T_pad" H 3650 3150 50  0001 C CNN
+F 2 "cap_touch_LPC804_NXP:Cap_T_pad_v1.1" H 3650 3150 50  0001 C CNN
 F 3 "~" H 3650 3150 50  0001 C CNN
 	1    3650 3150
@@
 F 0 "C5" H 4428 3196 50  0000 L CNN
 F 1 "CAPT" H 4428 3105 50  0000 L CNN
-F 2 "cap_touch_LPC804_NXP:Cap_T_pad" H 4250 3150 50  0001 C CNN
+F 2 "cap_touch_LPC804_NXP:Cap_T_pad_v1.1" H 4250 3150 50  0001 C CNN
 F 3 "~" H 4250 3150 50  0001 C CNN
 	1    4250 3150
