File: clock/clock.sch (KiCad schematic (older format))
At the start: 173 parts, among them J1 Conn_01x06_Female, P1 Conn_WallPlug, SW1 SW_Push, SW2 SW_Push, SW3 SW_Push, T1 120 to 12, U1 NPIC6C596A, U10 NPIC6C596A, U11 PIC18F45K20_44-PIN_TQFP, U2 NPIC6C596A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

Commit message: Setup gerbers
Parts:
- T1: footprint (none) -> TerminalBlock:TerminalBlock_bornier-2_P5.08mm
Changed lines of the file:
@@
 F 0 "T1" H 2100 1628 50  0000 C CNN
 F 1 "120 to 12" H 2100 1537 50  0000 C CNN
-F 2 "" H 2100 1250 50  0001 C CNN
+F 2 "TerminalBlock:TerminalBlock_bornier-2_P5.08mm" H 2100 1250 50  0001 C CNN
 F 3 "~" H 2100 1250 50  0001 C CNN
 	1    2100 1250
@@
 Text GLabel 5400 2850 0    50   Input ~ 0
 Minus
-Wire Wire Line
-	5400 2850 5500 2850
-Wire Wire Line
-	5500 2850 5550 2850
 Connection ~ 5500 2850
 Wire Wire Line
 	5500 2850 5550 2850
 Connection ~ 5550 2850
+Wire Wire Line
+	5400 2850 5550 2850
 $EndSCHEMATC
